Commit message: Add PatrickBot code changes

File: pwrs_description/urdf/spongebot.urdf.xacro (robot description, xacro)
@@ -48,5 +48,5 @@
   <xacro:property name="hub_dia" value="0.09652"/>
   <xacro:property name="tire_dia" value="0.1905"/>
-  <xacro:property name="tire_width" value="0.09525"/>
+  <xacro:property name="tire_width" value="0.05"/>
   <xacro:property name="hex_hub_depth" value="0.01445"/>
   <xacro:property name="wheel_mass" value="0.10"/> <!-- TODO: Measure actual -->
@@ -183,7 +183,4 @@
       </joint>
       <actuator name="${lr_prefix}_${fr_prefix}_axle_act">
-        <!-- This hardwareInterface element exists for compatibility
-             with ROS Hydro. -->
-        <hardwareInterface>EffortJointInterface</hardwareInterface>
         <mechanicalReduction>1</mechanicalReduction>
       </actuator>
@@ -193,5 +190,5 @@
         <origin xyz="0 0 0"/>
         <geometry>
-          <mesh filename="file:///C:/tfs/ros/pwrs_ws/install/share/pwrs_description/urdf/CarTyre_${lr_prefix}.stl" scale="0.01 0.01 0.01" />
+          <mesh filename="package://pwrs_description/urdf/CarTyre_${lr_prefix}.stl" scale="0.01 0.01 0.01" />
         </geometry>
         <material name="tire_mat"/>
@@ -230,7 +227,4 @@
       </joint>
       <actuator name="${lr_prefix}_steering_act">
-        <!-- This hardwareInterface element exists for compatibility
-             with ROS Hydro. -->
-        <hardwareInterface>EffortJointInterface</hardwareInterface>
         <mechanicalReduction>1</mechanicalReduction>
       </actuator>
@@ -267,5 +261,5 @@
       <origin xyz="0 0 ${-chassis_height / 2}"/>
       <geometry>
-        <mesh filename="file:///C:/tfs/ros/pwrs_ws/install/share/pwrs_description/urdf/CarBody.stl" scale="0.01 0.01 0.01" />
+        <mesh filename="package://pwrs_description/urdf/CarBody.stl" scale="0.01 0.01 0.01" />
       </geometry>
       <material name="chassis_mat"/>
@@ -287,4 +281,16 @@
     <child link="chassis"/>
   </joint>
+  <link name="imu_link"/>
+  <joint name="imu_joint" type="fixed">
+    <parent link="chassis"/>
+    <child link="imu_link"/>
+    <origin xyz="0 0 0.0" rpy="0 0 0"/>
+  </joint>
+  <link name="odom_link"/>
+  <joint name="odom_joint" type="fixed">
+    <parent link="chassis"/>
+    <child link="odom_link"/>
+    <origin xyz="0 0 -0.24" rpy="0 0 0"/>
+  </joint>
   <!-- Batteries -->
   <xacro:battery prefix="left" reflect="1"/>
